File: IGN6.kicad_sch (KiCad schematic)
At the start: 12 parts

Commit message: stabil jr.
Parts:
- removed F10, F9: 50mA, Fuse:Fuse_0603_1608Metric, symbol Device:Polyfuse
- removed R27, R28: 0, hellen-one-common:R0603, symbol hellen-one-common:Res
- renumbered F6 to F11, F5 to F12, F7 to F13, F8 to F14, R20 to R11, R21 to R12, R22 to R13, R26 to R14
Other:
- note removed: "Remove R20-R22, R26-R28, and install Q7-Q12 for use with dumb coils"
