File: INJ6.kicad_sch (KiCad schematic)
At the start: 9 parts, among them U10 VNLD5160TR-E, U11 VNLD5160TR-E, U9 VNLD5160TR-E

Commit message: stabil jr.
Parts:
- removed R30 (x2): 4.7k, hellen-one-common:R0603, symbol hellen-one-common:Res
- removed U11: VNLD5160TR-E, Package_SO:SOIC-8_3.9x4.9mm_P1.27mm, symbol chips:VNLD5160
- renumbered R30 to R21, R30 to R22, R30 to R23, R30 to R24
Connections:
- no-connect marks 6 -> 4
