File: LS_HOT.kicad_sch (KiCad schematic)
At the start: 3 parts, among them U6 VNLD5160TR-E

Commit message: stabil jr.
Parts:
- renumbered R30 to R5, R30 to R6, U6 to U3
Changed lines of the file:
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@@
 		(on_board yes)
 		(dnp no)
-		(property "Reference" "#PWR0140"
+		(property "Reference" "#PWR024"
 			(at 129.54 102.87 0)
 			(effects
@@
 		)
 		(instances
-			(project "uaefi"
-				(path "/ac264c30-3e9a-4be2-b97a-9949b68bd497/c1e0fc38-44a5-4f4c-8a40-7ced112340c0"
-					(reference "#PWR0140")
+			(project "stabildaytona"
+				(path "/ac264c30-3e9a-4be2-b97a-9949b68bd497/48c489a8-99d9-428c-87a8-b1eeb5836df2"
+					(reference "#PWR024")
+					(unit 1)
+				)
+				(path "/ac264c30-3e9a-4be2-b97a-9949b68bd497/c1e0fc38-44a5-4f4c-8a40-7ced112340c0"
+					(reference "#PWR0101")
+					(unit 1)
+				)
+				(path "/ac264c30-3e9a-4be2-b97a-9949b68bd497/eaaf5216-1f1d-4979-a2cc-7a4c348e8094"
+					(reference "#PWR05")
 					(unit 1)
 				)
@@
 		(dnp no)
 		(fields_autoplaced yes)
-		(property "Reference" "U6"
+		(property "Reference" "U3"
 			(at 146.05 78.74 0)
 			(effects
@@
 		)
 		(instances
-			(project "uaefi"
-				(path "/ac264c30-3e9a-4be2-b97a-9949b68bd497/c1e0fc38-44a5-4f4c-8a40-7ced112340c0"
-					(reference "U6")
+			(project "stabildaytona"
+				(path "/ac264c30-3e9a-4be2-b97a-9949b68bd497/48c489a8-99d9-428c-87a8-b1eeb5836df2"
+					(reference "U3")
+					(unit 1)
+				)
+				(path "/ac264c30-3e9a-4be2-b97a-9949b68bd497/c1e0fc38-44a5-4f4c-8a40-7ced112340c0"
+					(reference "U1")
+					(unit 1)
+				)
+				(path "/ac264c30-3e9a-4be2-b97a-9949b68bd497/eaaf5216-1f1d-4979-a2cc-7a4c348e8094"
+					(reference "U2")
 					(unit 1)
 				)
@@
 		(on_board yes)
 		(dnp no)
-		(property "Reference" "#PWR035"
+		(property "Reference" "#PWR027"
 			(at 180.34 102.87 0)
 			(effects
@@
 		)
 		(instances
-			(project "alphax_8ch"
-				(path "/63d2dd9f-d5ff-4811-a88d-0ba932475460"
-					(reference "#PWR035")
-					(unit 1)
-				)
-				(path "/63d2dd9f-d5ff-4811-a88d-0ba932475460/9f286606-17ad-4292-b95a-d7d4de96430a"
-					(reference "#PWR0165")
-					(unit 1)
-				)
-			)
-			(project "uaefi"
-				(path "/ac264c30-3e9a-4be2-b97a-9949b68bd497/c1e0fc38-44a5-4f4c-8a40-7ced112340c0"
-					(reference "#PWR094")
+			(project "stabildaytona"
+				(path "/ac264c30-3e9a-4be2-b97a-9949b68bd497/48c489a8-99d9-428c-87a8-b1eeb5836df2"
+					(reference "#PWR027")
+					(unit 1)
+				)
+				(path "/ac264c30-3e9a-4be2-b97a-9949b68bd497/c1e0fc38-44a5-4f4c-8a40-7ced112340c0"
+					(reference "#PWR0103")
+					(unit 1)
+				)
+				(path "/ac264c30-3e9a-4be2-b97a-9949b68bd497/eaaf5216-1f1d-4979-a2cc-7a4c348e8094"
+					(reference "#PWR09")
 					(unit 1)
 				)
@@
 		(on_board yes)
 		(dnp no)
-		(property "Reference" "#PWR035"
+		(property "Reference" "#PWR025"
 			(at 168.91 107.95 0)
 			(effects
@@
 		)
 		(instances
-			(project "alphax_8ch"
-				(path "/63d2dd9f-d5ff-4811-a88d-0ba932475460"
-					(reference "#PWR035")
-					(unit 1)
-				)
-				(path "/63d2dd9f-d5ff-4811-a88d-0ba932475460/9f286606-17ad-4292-b95a-d7d4de96430a"
-					(reference "#PWR0165")
-					(unit 1)
-				)
-			)
-			(project "uaefi"
-				(path "/ac264c30-3e9a-4be2-b97a-9949b68bd497/c1e0fc38-44a5-4f4c-8a40-7ced112340c0"
-					(reference "#PWR095")
+			(project "stabildaytona"
+				(path "/ac264c30-3e9a-4be2-b97a-9949b68bd497/48c489a8-99d9-428c-87a8-b1eeb5836df2"
+					(reference "#PWR025")
+					(unit 1)
+				)
+				(path "/ac264c30-3e9a-4be2-b97a-9949b68bd497/c1e0fc38-44a5-4f4c-8a40-7ced112340c0"
+					(reference "#PWR0102")
+					(unit 1)
+				)
+				(path "/ac264c30-3e9a-4be2-b97a-9949b68bd497/eaaf5216-1f1d-4979-a2cc-7a4c348e8094"
+					(reference "#PWR07")
 					(unit 1)
 				)
@@
 		(on_board yes)
 		(dnp no)
-		(property "Reference" "R30"
+		(property "Reference" "R5"
 			(at 177.8 91.44 0)
 			(effects
@@
 		)
 		(instances
-			(project "alphax_8ch"
-				(path "/63d2dd9f-d5ff-4811-a88d-0ba932475460"
-					(reference "R30")
-					(unit 1)
-				)
-				(path "/63d2dd9f-d5ff-4811-a88d-0ba932475460/9f286606-17ad-4292-b95a-d7d4de96430a"
-					(reference "R68")
-					(unit 1)
-				)
-			)
-			(project "uaefi"
-				(path "/ac264c30-3e9a-4be2-b97a-9949b68bd497/c1e0fc38-44a5-4f4c-8a40-7ced112340c0"
-					(reference "R15")
+			(project "stabildaytona"
+				(path "/ac264c30-3e9a-4be2-b97a-9949b68bd497/48c489a8-99d9-428c-87a8-b1eeb5836df2"
+					(reference "R5")
+					(unit 1)
+				)
+				(path "/ac264c30-3e9a-4be2-b97a-9949b68bd497/c1e0fc38-44a5-4f4c-8a40-7ced112340c0"
+					(reference "R1")
+					(unit 1)
+				)
+				(path "/ac264c30-3e9a-4be2-b97a-9949b68bd497/eaaf5216-1f1d-4979-a2cc-7a4c348e8094"
+					(reference "R3")
 					(unit 1)
 				)
@@
 		(on_board yes)
 		(dnp no)
-		(property "Reference" "R30"
+		(property "Reference" "R6"
 			(at 166.37 96.52 0)
 			(effects
@@
 		)
 		(instances
-			(project "alphax_8ch"
-				(path "/63d2dd9f-d5ff-4811-a88d-0ba932475460"
-					(reference "R30")
-					(unit 1)
-				)
-				(path "/63d2dd9f-d5ff-4811-a88d-0ba932475460/9f286606-17ad-4292-b95a-d7d4de96430a"
-					(reference "R68")
-					(unit 1)
-				)
-			)
-			(project "uaefi"
-				(path "/ac264c30-3e9a-4be2-b97a-9949b68bd497/c1e0fc38-44a5-4f4c-8a40-7ced112340c0"
-					(reference "R16")
-					(unit 1)
-				)
+			(project "stabildaytona"
+				(path "/ac264c30-3e9a-4be2-b97a-9949b68bd497/48c489a8-99d9-428c-87a8-b1eeb5836df2"
+					(reference "R6")
+					(unit 1)
+				)
+				(path "/ac264c30-3e9a-4be2-b97a-9949b68bd497/c1e0fc38-44a5-4f4c-8a40-7ced112340c0"
+					(reference "R2")
+					(unit 1)
+				)
+				(path "/ac264c30-3e9a-4be2-b97a-9949b68bd497/eaaf5216-1f1d-4979-a2cc-7a4c348e8094"
+					(reference "R4")
+					(unit 1)
+				)
