File: MAP.kicad_sch (KiCad schematic)
At the start: 2 parts

Commit message: stabil jr.
Parts:
- MAP1: value MPXH6400A -> GZP6869D200KPP; LCSC C511770 -> C3038053
Changed lines of the file:
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@@
 			)
 		)
-		(property "Value" "MPXH6400A"
+		(property "Value" "GZP6869D200KPP"
 			(at 123.19 54.61 0)
 			(effects
@@
 			)
 		)
-		(property "Datasheet" ""
+		(property "Datasheet" "Sencoch Semiconductor"
 			(at 119.38 64.77 0)
 			(effects
@@
 			)
 		)
-		(property "Description" ""
+		(property "Description" "0Kpa~200Kpa I2C SOP-8 Pressure Sensors ROHS"
 			(at 119.38 64.77 0)
 			(effects
@@
 			)
 		)
-		(property "LCSC" "C511770"
+		(property "LCSC" "C3038053"
 			(at 119.38 64.77 0)
 			(effects
@@
 			(project "uaefi"
 				(path "/ac264c30-3e9a-4be2-b97a-9949b68bd497/7f618b1f-fe11-49db-a473-d0b521b1fa4f"
-					(reference "C27")
-					(unit 1)
-				)
+					(reference "C1")
+					(unit 1)
+				)
