File: stabildaytona.kicad_sch (KiCad schematic)
At the start: 22 parts, among them M1 Module-power_12and5V-0.2, M3 Module-knock-0.2, M4 Module-vr-max9924-0.1

Commit message: v1 tam test
Parts:
- removed G1: RUSEFI_LOGO, kicad6-libraries:rusefi_logo, symbol rusefi_logo:RUSEFI_LOGO
- removed G2: LOGO, hellen-one-common:LOGO, symbol hellen-one-common:LOGO
- BLUETOOTH1: LCSC (none) -> C22438154
- SAGSOKET1, SOLSOKET1: LCSC (none) -> C19630948
- USB1: LCSC (none) -> C265289
Connections:
- net GND: now also SAGSOKET1.18 (Pin_18), SAGSOKET1.20 (Pin_20), SAGSOKET1.22 (Pin_22)
Changed lines of the file:
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@@
 	(wire
 		(pts
-			(xy 91.44 389.89) (xy 105.41 389.89)
-		)
-		(stroke
-			(width 0)
-			(type default)
-		)
-	)
-	(wire
-		(pts
 			(xy 153.67 175.26) (xy 162.56 175.26)
 		)
@@
 	)
 	(label "VR_MAX9924-"
-		(at 93.98 389.89 0)
+		(at 105.41 389.89 180)
 		(fields_autoplaced yes)
 		(effects
@@
 				(size 1.27 1.27)
 			)
-			(justify left bottom)
+			(justify right bottom)
 		)
 	)
@@
 	)
 	(symbol
-		(lib_id "hellen-one-common:LOGO")
-		(at 189.23 377.19 0)
-		(unit 1)
-		(exclude_from_sim no)
-		(in_bom yes)
-		(on_board yes)
-		(dnp no)
-		(fields_autoplaced yes)
-		(property "Reference" "G2"
-			(at 189.23 379.8062 0)
-			(effects
-				(font
-					(size 1.524 1.524)
-				)
-				(hide yes)
-			)
-		)
-		(property "Value" "LOGO"
-			(at 189.23 374.5738 0)
-			(effects
-				(font
-					(size 1.524 1.524)
-				)
-				(hide yes)
-			)
-		)
-		(property "Footprint" "hellen-one-common:LOGO"
-			(at 190.5 382.27 0)
-			(effects
-				(font
-					(size 1.27 1.27)
-				)
-				(hide yes)
-			)
-		)
-		(property "Datasheet" ""
-			(at 176.53 377.19 0)
-			(effects
-				(font
-					(size 1.27 1.27)
-				)
-				(hide yes)
-			)
-		)
-		(property "Description" ""
-			(at 189.23 377.19 0)
-			(effects
-				(font
-					(size 1.27 1.27)
-				)
-				(hide yes)
-			)
-		)
-		(instances
-			(project "uaefi"
-				(path "/ac264c30-3e9a-4be2-b97a-9949b68bd497"
-					(reference "G2")
-					(unit 1)
-				)
-			)
-		)
-	)
-	(symbol
 		(lib_id "power:GND")
 		(at 105.41 397.51 270)
@@
 	)
 	(symbol
-		(lib_id "rusefi_logo:RUSEFI_LOGO")
-		(at 181.61 382.27 0)
+		(lib_id "power:GNDA")
+		(at 48.26 90.17 270)
+		(mirror x)
 		(unit 1)
 		(exclude_from_sim no)
@@
 		(on_board yes)
 		(dnp no)
-		(fields_autoplaced yes)
-		(property "Reference" "G1"
-			(at 181.61 384.8862 0)
+		(property "Reference" "#PWR022"
+			(at 41.91 90.17 0)
 			(effects
 				(font
-					(size 1.524 1.524)
+					(size 1.27 1.27)
 				)
 				(hide yes)
 			)
 		)
-		(property "Value" "RUSEFI_LOGO"
-			(at 181.61 379.6538 0)
+		(property "Value" "GND"
+			(at 42.6656 90.0557 90)
 			(effects
 				(font
-					(size 1.524 1.524)
+					(size 1.27 1.27)
 				)
-				(hide yes)
 			)
 		)
-		(property "Footprint" "kicad6-libraries:rusefi_logo"
-			(at 181.61 382.27 0)
+		(property "Footprint" ""
+			(at 48.26 90.17 0)
 			(effects
 				(font
@@
 		)
 		(property "Datasheet" ""
-			(at 181.61 382.27 0)
+			(at 48.26 90.17 0)
 			(effects
 				(font
@@
 		)
 		(property "Description" ""
-			(at 181.61 382.27 0)
+			(at 48.26 90.17 0)
 			(effects
 				(font
@@
 			)
 		)
+		(pin "1"
+		)
 		(instances
-			(project "uaefi"
+			(project "stabildaytona"
 				(path "/ac264c30-3e9a-4be2-b97a-9949b68bd497"
-					(reference "G1")
+					(reference "#PWR022")
 					(unit 1)
 				)
@@
 	)
 	(symbol
+		(lib_id "power:GNDA")
+		(at 48.26 95.25 270)
+		(mirror x)
+		(unit 1)
+		(exclude_from_sim no)
+		(in_bom yes)
+		(on_board yes)
+		(dnp no)
+		(property "Reference" "#PWR035"
+			(at 41.91 95.25 0)
+			(effects
+				(font
+					(size 1.27 1.27)
+				)
+				(hide yes)
+			)
+		)
+		(property "Value" "GND"
+			(at 42.6656 95.1357 90)
+			(effects
+				(font
+					(size 1.27 1.27)
+				)
+			)
+		)
+		(property "Footprint" ""
+			(at 48.26 95.25 0)
+			(effects
+				(font
+					(size 1.27 1.27)
+				)
+				(hide yes)
+			)
+		)
+		(property "Datasheet" ""
+			(at 48.26 95.25 0)
+			(effects
+				(font
+					(size 1.27 1.27)
+				)
+				(hide yes)
+			)
+		)
+		(property "Description" ""
+			(at 48.26 95.25 0)
+			(effects
+				(font
+					(size 1.27 1.27)
+				)
+				(hide yes)
+			)
+		)
+		(pin "1"
+		)
+		(instances
+			(project "stabildaytona"
+				(path "/ac264c30-3e9a-4be2-b97a-9949b68bd497"
+					(reference "#PWR035")
+					(unit 1)
+				)
+			)
+		)
+	)
+	(symbol
 		(lib_id "Connector_Generic:Conn_02x20_Counter_Clockwise")
 		(at 53.34 135.89 0)
@@
 			)
 		)
+		(property "LCSC" "C19630948"
+			(at 53.34 135.89 0)
+			(effects
+				(font
+					(size 1.27 1.27)
+				)
+				(hide yes)
+			)
+		)
 		(pin "17"
 		)
@@
 			)
 		)
+		(property "LCSC" "C19630948"
+			(at 53.34 69.85 0)
+			(effects
+				(font
+					(size 1.27 1.27)
+				)
+				(hide yes)
+			)
+		)
 		(pin "17"
 		)
@@
 	)
 	(symbol
+		(lib_id "power:GNDA")
+		(at 60.96 92.71 90)
+		(mirror x)
+		(unit 1)
+		(exclude_from_sim no)
+		(in_bom yes)
+		(on_board yes)
+		(dnp no)
+		(property "Reference" "#PWR036"
+			(at 67.31 92.71 0)
+			(effects
+				(font
+					(size 1.27 1.27)
+				)
+				(hide yes)
+			)
+		)
+		(property "Value" "GND"
+			(at 66.5544 92.8243 90)
+			(effects
+				(font
+					(size 1.27 1.27)
+				)
+			)
+		)
+		(property "Footprint" ""
+			(at 60.96 92.71 0)
+			(effects
+				(font
+					(size 1.27 1.27)
+				)
+				(hide yes)
+			)
+		)
+		(property "Datasheet" ""
+			(at 60.96 92.71 0)
+			(effects
+				(font
+					(size 1.27 1.27)
+				)
+				(hide yes)
+			)
+		)
+		(property "Description" ""
+			(at 60.96 92.71 0)
+			(effects
+				(font
+					(size 1.27 1.27)
+				)
+				(hide yes)
+			)
+		)
+		(pin "1"
+		)
+		(instances
+			(project "stabildaytona"
+				(path "/ac264c30-3e9a-4be2-b97a-9949b68bd497"
+					(reference "#PWR036")
+					(unit 1)
+				)
+			)
+		)
+	)
+	(symbol
 		(lib_id "power:+12V")
 		(at 194.31 340.36 0)
@@
 			)
 		)
+		(property "LCSC" "C22438154"
+			(at 240.03 339.09 0)
+			(effects
+				(font
+					(size 1.27 1.27)
+				)
+				(hide yes)
+			)
+		)
 		(pin "4"
 		)
@@
 			)
 		)
+		(property "LCSC" "C265289"
+			(at 266.7 339.09 0)
+			(effects
+				(font
+					(size 1.27 1.27)
+				)
+				(hide yes)
+			)
+		)
 		(pin "3"
 		)
@@
 				)
 			)
-			(project "stabil-daytona"
+			(project "stabildaytona"
 				(path "/ac264c30-3e9a-4be2-b97a-9949b68bd497"
 					(page "2")
@@
 		)
 		(instances
-			(project "stabil-daytona"
+			(project "stabildaytona"
 				(path "/ac264c30-3e9a-4be2-b97a-9949b68bd497"
 					(page "10")
@@
 		)
 		(instances
-			(project "stabil-daytona"
+			(project "stabildaytona"
 				(path "/ac264c30-3e9a-4be2-b97a-9949b68bd497"
 					(page "8")
@@
 		)
 		(instances
-			(project "stabil-daytona"
+			(project "stabildaytona"
 				(path "/ac264c30-3e9a-4be2-b97a-9949b68bd497"
 					(page "9")
@@
 		)
 		(instances
-			(project "stabil-daytona"
+			(project "stabildaytona"
 				(path "/ac264c30-3e9a-4be2-b97a-9949b68bd497"
 					(page "3")
@@
 				)
 			)
-			(project "stabil-daytona"
+			(project "stabildaytona"
 				(path "/ac264c30-3e9a-4be2-b97a-9949b68bd497"
 					(page "4")
@@
 		)
 		(instances
-			(project "stabil-daytona"
+			(project "stabildaytona"
 				(path "/ac264c30-3e9a-4be2-b97a-9949b68bd497"
 					(page "6")
@@
 		)
 		(instances
-			(project "stabil-daytona"
+			(project "stabildaytona"
 				(path "/ac264c30-3e9a-4be2-b97a-9949b68bd497"
 					(page "9")

Commit message: stabil jr.
Parts:
- removed CAN1: Module-can-0.1, hellen-one-can-0.1:can, symbol hellen-one-can-0.1:Module-can-0.1
- removed F1, F6 (x2): 12H1500D, hellen-one-common:PAD-1206-PAD, symbol hellen-one-common:Fuse-Pad-Pad
- removed M3: Module-knock-0.2, hellen-one-knock-0.2:knock, symbol hellen-one-knock-0.2:Module-knock-0.2
- removed R30: 0, hellen-one-common:R0603, symbol hellen-one-common:Res
- removed SAGSOKET1, SOLSOKET1: Conn_02x20_Counter_Clockwise, Connector_PinHeader_2.54mm:PinHeader_2x20_P2.54mm_Vertical, symbol Connector_Generic:Conn_02x20_Counter_Clockwise
- added J1: Conn_01x24, Connector:24pin, symbol Connector_Generic:Conn_01x24
- added J2: Conn_01x20, Connector_TE-Connectivity:TE_2-826576-0_1x20_P3.96mm_Vertical, symbol Connector_Generic:Conn_01x20
- added R41, R42: 2.7K, hellen-one-common:R0805, symbol hellen-one-common:Res
- added R43: 10K, hellen-one-common:R0805, symbol hellen-one-common:Res
- renumbered R5 to R31, R7 to R32, R8 to R33, R3 to R7, R2 to R8, R4 to R9, MCU1 to İŞLEMC1
Connections:
- net +5VP is gone; now on net +5V: M1.V4 (5VP)
- net IN_VIGN is gone; now on net +12V_RAW: M1.V2 (IN_VIGN)
- net +12V: now also R43.1
- net +12V_RAW: now also J1.8 (Pin_8)
- net +5V: now also J1.1 (Pin_1)
- net +5VA: now also J2.18 (Pin_18), R41.1, R42.1
- net BT_RX: now also J2.16 (Pin_16)
- net BT_TX: now also J2.17 (Pin_17)
- net CAN1+: now also J2.7 (Pin_7)
- net CAN1-: now also J2.8 (Pin_8)
- net GND: now also J1.24 (Pin_24), J2.19 (Pin_19), J2.20 (Pin_20)
- net GNDA: now also J1.16 (Pin_16)
- net IN_BUTTON1: now also J2.4 (Pin_4)
- net IN_BUTTON2: now also J2.5 (Pin_5)
- net IN_BUTTON3: now also J2.6 (Pin_6)
- net IN_CLT: now also J1.14 (Pin_14), R42.2
- net IN_HALL1: now also J1.23 (Pin_23)
- net IN_HALL2: now also J2.1 (Pin_1)
- net IN_HALL3: now also J2.2 (Pin_2)
- net IN_IAT: now also J1.15 (Pin_15), R41.2
- net VR_MAX9924+: now also J1.6 (Pin_6)
- net VR_MAX9924-: now also J1.7 (Pin_7)
- net ADC3: no longer names the net of İŞLEMC1.S15 (IN_KNOCK_(PA2))
- net DC1_DIR: no longer names the net of İŞLEMC1.E21 (OUT_PWM4_(PC8))
- net DC1_DIS: no longer names the net of İŞLEMC1.E8 (SPI2_MISO_(PB14))
- net DC1_PWM: no longer names the net of İŞLEMC1.E20 (OUT_PWM3_(PC7))
- net DC2_DIR: no longer names the net of İŞLEMC1.E9 (SPI2_MOSI_(PB15))
- net DC2_DIS: no longer names the net of İŞLEMC1.N4 (USBID_(PA10))
- net DC2_PWM: no longer names the net of İŞLEMC1.E22 (OUT_PWM5_(PC9))
- net EGT/SPI_CS: no longer names the net of İŞLEMC1.N9 (SPI3_CS_(PA15))
- net EGT/SPI_SCK: no longer names the net of İŞLEMC1.N10 (SPI3_SCK_(PC10))
- net EGT/SPI_SO: no longer names the net of İŞLEMC1.N11 (SPI3_MISO_(PC11))
- net IGN1 renamed BOBIN/IN1
- net IGN2 renamed BOBIN/IN2
- net IGN3 renamed BOBIN/IN3
- net IGN4 renamed BOBIN/IN4
- net IGN5: no longer names the net of İŞLEMC1.W6 (IGN5_(PE2))
- net IGN6: no longer names the net of İŞLEMC1.W5 (IGN6_(PB8))
- net INJ1 renamed ENJEKTOR/IN1
- net INJ2 renamed ENJEKTOR/IN2
- net INJ3 renamed ENJEKTOR/IN3
- net INJ4 renamed ENJEKTOR/IN4
- net INJ5: no longer names the net of İŞLEMC1.E13 (OUT_INJ5_(PD2))
- net INJ6: no longer names the net of İŞLEMC1.E12 (OUT_INJ6_(PA8))
- net IN_AUX1 renamed ANALOG 3
- net ANALOG 3: now also J2.9 (Pin_9)
- net IN_AUX2 renamed ANALOG 4
- net ANALOG 4: now also J2.10 (Pin_10)
- net IN_AUX3 renamed ANALOG 8
- net ANALOG 8: now also J2.14 (Pin_14)
- net IN_FLEX renamed IN_HALL4
- net IN_HALL4: now also J2.3 (Pin_3)
- net IN_MAP renamed ANALOG 5
- net ANALOG 5: now also J2.11 (Pin_11)
- net IN_PPS1 renamed ANALOG 2
- net ANALOG 2: now also J1.17 (Pin_17)
- net IN_PPS2 renamed ANALOG 7
- net ANALOG 7: now also J2.13 (Pin_13)
- net IN_TPS1 renamed ANALOG 1
- net ANALOG 1: now also J1.9 (Pin_9)
- net IN_TPS2 renamed ANALOG 6
- net ANALOG 6: now also J2.12 (Pin_12)
- net LS1 renamed AUX GROUP 2/IN1
- net LS2 renamed AUX GROUP 2/IN2
- net LS3 renamed AUX GROUP 3/IN1
- net LS4 renamed AUX GROUP 3/IN2
- net LS_HOT1 renamed AUX GROUP 1/IN1
- net LS_HOT2 renamed AUX GROUP 1/IN2
- net MCU-CAN2RX: no longer names the net of İŞLEMC1.E6 (SPI2_CS_/_CAN2_RX_(PB12))
- net MCU-CAN2TX: no longer names the net of İŞLEMC1.E7 (SPI2_SCK_/_CAN2_TX_(PB13))
- new net BOBİN 1: J1.2 (Pin_2)
- new net BOBİN 2: J1.3 (Pin_3)
- new net BOBİN 3: J1.4 (Pin_4)
- new net BOBİN 4: J1.5 (Pin_5)
- new net ENJEKTÖR 1: J1.10 (Pin_10)
- new net ENJEKTÖR 2: J1.11 (Pin_11)
- new net ENJEKTÖR 3: J1.12 (Pin_12)
- new net ENJEKTÖR 4: J1.13 (Pin_13)
- new net ÇIKIŞ 1: J1.18 (Pin_18), R43.2
- new net ÇIKIŞ 2: J1.19 (Pin_19)
- new net ÇIKIŞ 3: J1.20 (Pin_20)
- new net ÇIKIŞ 4: J1.21 (Pin_21)
- new net ÇIKIŞ 5: J1.22 (Pin_22)
- new net ÇIKIŞ 6: J2.15 (Pin_15)
- no-connect marks 19 -> 36
Other:
- sheet Ignition renamed BOBIN
- sheet Injector renamed ENJEKTOR
- sheet LS HOT renamed AUX GROUP 1
- removed sheet DC Driver 1
- removed sheet DC Driver 2
- removed sheet EGT
- removed sheet LS
- added sheet AUX GROUP 2 (LS_HOT.kicad_sch)
- added sheet AUX GROUP 3 (LS_HOT.kicad_sch)
- sheet BOBIN ports: added none; removed IN5, IN6, OUT5, OUT6
- sheet ENJEKTOR ports: added none; removed IN5, IN6, OUT5, OUT6
- note removed: "3.5A MAX Always hot capable"
- note removed: "3.5A MAX Solenoid load capable"
- moved on the sheet: BLUETOOTH1, M1, M4, R9
